Commit message: first point

File: ros2_iiwa/iiwa_description/urdf/iiwa.urdf.xacro (robot description, xacro)
@@ -225,4 +225,6 @@
       <axis xyz="0 0 0"/>
   </joint>
+  <xacro:property name="use_vision" value="$(arg use_vision)" />
+  <xacro:if value="${use_vision}">
   <xacro:include filename="$(find iiwa_description)/urdf/arm_camera.xacro" />
     <joint name="camera_joint" type="fixed">
@@ -240,4 +242,5 @@
   </link>
   <xacro:arm_camera name="camera" link_reference="camera_link"/>
+  </xacro:if>
   </xacro:macro>
 </robot>
